File: laika-bess-hw/laika-bess-hw.kicad_sch (KiCad schematic)
At the start: 0 parts

Commit message: Replace the on-board autoencoder with threshold rules
Detection now uses explicit thresholds on gas, enclosure pressure and air
temperature, decided on the module (rules.h, see DETECTION.md):
- per channel: gas <= 60/35 % of its clean-air level, |dP| >= 50/200 Pa,
  TMP117 >= 45/60 degC, rise >= 1 degC/min, gas <= 80 % for an hour (leak);
- possible battery event = two channels within a minute, or 60 degC.
  One channel alone is usually an everyday disturbance (people, a door,
  sun), so it is a warning, not the alarm.

Replaying 10.5 h of real logs: no battery-event alarms; gas and pressure
disturbances stayed single-channel. The autoencoder (in history up to
349c6ce) sat in constant alarm once the air was cleaner than its training
night; whether it is the better approach will be decided after real testing.

Protocol v4 carries the rule bits in place of the autoencoder score. The
Pi dashboard shows the module's verdict (battery event check panel) and
reads the thresholds from rules.h at deploy, so the two can't disagree.
Also: tools/check_rules.py (replay), tools/rules_json.py, DETECTION.md,
logger fix for fields of older frame versions.

Co-Authored-By: Claude Opus 5.5 <noreply@anthropic.com>
Parts:
- added BT1: Battery_Cell, symbol Device:Battery_Cell
- added J1: (no value), symbol Connector:RPI-HAL
- added U1: (no value), symbol MCU_AnalogDevices:MAX32630FTHR#
- added U2: (no value), symbol Sensor_Gas:BME688
- added U3: (no value), symbol Sensor_Temperature:TMP117
- added U4: ABPxxxxxxxxx0, symbol Sensor_Pressure:ABPxxxxxxxxx0
Connections:
- new net +3V3: U1. (P3_4), U2. (CS), U3. (ADDR), U4.2 (VCC)
- new net +BATT: BT1.1 (+), U1. (P3_4)
- new net -BATT: BT1.2 (-), U1. (P3_4)
- new net GND: J1. (6/GND), U1. (P3_4), U2. (CS), U3. (ADDR), U4.1 (GND)
- new net PI_RX: J1. (6/GND), U1. (P3_4)
- new net PI_TX: J1. (6/GND), U1. (P3_4)
- new net SCL: U1. (P3_4), U2. (CS), U3. (ADDR), U4.6 (SCL)
- new net SDA: U1. (P3_4), U2. (CS), U3. (ADDR), U4.5 (SDA)
- no-connect marks 0 -> 26
Other:
- company: (none) ->           Laika IIoT Technologies Pvt. Ltd.
- title: (none) -> Pack Agnostic Thermal Runaway Detection for BESS
